File: kicad/conch/conch.kicad_pcb (KiCad board)
At the start: 2 copper layers, 52 x 36 mm, 19 parts, among them J1 Conn_01x02_Socket, J2 TouchConnector, J3 UARTConnector, J4 SWIMConnector, M1 Motor_DC, Q1 AO3400A, SW1 SW_Push, U1 STM8S001J3M, U2 LMV321, U3 AMS1117

Commit message: feat(kicad):new cad
Parts:
- added C4: 470uF, Capacitor_THT:CP_Radial_D6.3mm_P2.50mm, F.Cu at (169.2, 69.6)
- added C5: 100uF, Capacitor_THT:CP_Radial_D5.0mm_P2.50mm, F.Cu at (123.5, 75.6)
- moved U3 6.41 mm to (124.6, 86.6)
- moved J3 2.50 mm to (160.6, 68.6)
- moved J4 1.95 mm to (146.6, 68.6)
- moved SW1 0.75 mm to (135.3, 68.6)
Connections:
- D2 pad 1: VCC -> +BATT
- J1 pad 1: Net-(J1-Pin_1) -> +BATT
- J1 pad 2: Net-(J1-Pin_2) -> GNDPWR
- M1 pad 1: VCC -> +BATT
- Q1 pad 2: GND -> GNDPWR
- R2 pad 1: VCC -> +BATT
- R4 pad 2: GND -> GNDPWR
- SW1 pad 1: Net-(J1-Pin_2) -> GNDPWR
- U2 pad 5: VCC -> +BATT
- U3 pad 3: Net-(J1-Pin_1) -> +BATT
Routing:
- net +BATT: track 0.00 -> 106.2 mm, vias 0 -> 1
- net GNDPWR: track 0.00 -> 40.4 mm, vias 0 -> 1
- net VCC: track 132.9 -> 97.1 mm, vias 2 -> 0
- net Net-(J1-Pin_2): track 13.9 -> 0.00 mm
- net Net-(D2-A): track 16.8 -> 27.1 mm
- net Net-(J1-Pin_1): track 10.0 -> 0.00 mm
- net DEBUG_UART_TX/SWIM: track 37.4 -> 44.3 mm
- net GND: vias 2 -> 1
Other:
- board text added: "2026-04-04 Conch v3.0 by jucat"
- board text removed: "Conch v2.0 by LMR"

Commit message: fix(conch):conch sch v4
Parts:
- added C6: 0.1uF, Capacitor_SMD:C_0603_1608Metric, F.Cu at (124.0, 91.1)
- added D3: 1N5822, Diode_SMD:D_SMA, F.Cu at (125.5, 75.6)
- added L1: 10uH, Inductor_SMD:L_0603_1608Metric, F.Cu at (124.3, 80.9)
- moved C4 34.9 mm to (135.2, 77.6)
- moved M1 29.7 mm to (137.7, 67.5), turned to 180 degrees
- moved J4 22.6 mm to (165.7, 80.6), turned to 90 degrees
- moved U1 16.8 mm to (155.5, 84.5)
- moved C2 15.6 mm to (148.5, 83.9)
- moved C3 15.5 mm to (148.4, 86.0), turned to 0 degrees
- moved C1 15.4 mm to (148.5, 88.4), turned to 180 degrees
- moved R3 12.8 mm to (140.1, 93.2), turned to 180 degrees
- moved D2 12.4 mm to (150.2, 75.6), turned to 180 degrees
- moved SW1 12.4 mm to (147.7, 67.5)
- moved C5 10.9 mm to (125.1, 86.4), turned to 180 degrees
- moved R2 9.65 mm to (140.1, 89.6), turned to 0 degrees
- moved U3 9.07 mm to (132.6, 91.0)
- moved U2 8.60 mm to (140.0, 83.7), turned to 90 degrees
- moved Q1 7.83 mm to (155.8, 77.6)
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Connections:
- C5 pad 1: +BATT -> Net-(U3-VI)
- C5 pad 2: +BATT -> GND
- J1 pad 2: GNDPWR -> Net-(J1-Pin_2)
- Q1 pad 2: GNDPWR -> GND
- R4 pad 2: GNDPWR -> GND
- SW1 pad 1: GNDPWR -> Net-(J1-Pin_2)
- U2 pad 5: +BATT -> VCC
- U3 pad 3: +BATT -> Net-(U3-VI)
Routing:
- net +BATT: track 106.2 -> 0.00 mm, vias 1 -> 0
- net VCC: track 97.1 -> 0.00 mm
- net DEBUG_UART_TX/SWIM: track 44.3 -> 0.00 mm
- net GNDPWR: track 40.4 -> 0.00 mm, vias 1 -> 0
- net Net-(D2-A): track 27.1 -> 0.00 mm
- net TOUCH: track 22.9 -> 0.00 mm
- net MOTOR: track 12.3 -> 0.00 mm
- net BATTERY_V: track 10.7 -> 0.00 mm
- net Net-(U2-+): track 9.03 -> 0.00 mm
- net LED: track 5.13 -> 0.00 mm
- net Net-(D1-A): track 4.22 -> 0.00 mm
- net GND: track 4.16 -> 0.00 mm, vias 1 -> 0
- net Net-(U1-VCAP): track 2.54 -> 0.00 mm
- removed copper zone on B.Cu, net GND
- removed copper zone on F.Cu, net GND
Other:
- board text removed: "2026-04-04 Conch v3.0 by jucat"

Commit message: fix(conch):new pcb
Parts:
- added R5: 0, Resistor_SMD:R_0603_1608Metric, F.Cu at (143.8, 78.7)
- moved D2 8.59 mm to (141.6, 75.1)
- moved Q1 7.57 mm to (148.6, 79.7), turned to -90 degrees
- moved C4 4.75 mm to (134.0, 82.2)
- moved R4 4.50 mm to (148.1, 75.6)
- moved J4 1.61 mm to (164.7, 81.8)
- moved J2 1.43 mm to (164.7, 93.6)
- moved D3 1.00 mm to (125.5, 76.6)
- moved R2 1.00 mm to (140.1, 88.6)
- moved J3 0.89 mm to (163.0, 68.4)
- moved M1 0.89 mm to (137.5, 68.4)
- moved SW1 0.89 mm to (147.5, 68.4)
- moved J1 0.89 mm to (127.0, 68.4)
- moved C6 0.32 mm to (124.4, 91.1)
- moved C1 0.24 mm to (148.4, 88.6)
- moved U2 0.17 mm to (140.1, 83.6), turned to 180 degrees
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Connections:
- Q1 pad 2: GND -> GNDPWR
- R3 pad 2: GND -> GNDPWR
- R4 pad 2: GND -> GNDPWR
Routing:
- net VCC: track 0.00 -> 78.5 mm, vias 0 -> 4
- net +BATT: track 0.00 -> 50.0 mm
- net Net-(D2-A): track 0.00 -> 32.3 mm, vias 0 -> 2
- net Net-(J1-Pin_2): track 0.00 -> 25.3 mm
- net DEBUG_UART_TX/SWIM: track 0.00 -> 21.1 mm
- net Net-(U3-VI): track 0.00 -> 17.2 mm
- net MOTOR: track 0.00 -> 14.6 mm, vias 0 -> 2
- net BATTERY_V: track 0.00 -> 14.1 mm
- net Net-(U2-+): track 0.00 -> 8.58 mm
- net TOUCH: track 0.00 -> 8.18 mm
- net LED: track 0.00 -> 7.06 mm
- net Net-(D3-K): track 0.00 -> 4.31 mm
- net Net-(U1-VCAP): track 0.00 -> 4.12 mm
- net Net-(D1-A): track 0.00 -> 3.18 mm
- net GNDPWR: track 0.00 -> 0.41 mm, vias 0 -> 4
- added copper zone on B.Cu, net GND
- added copper zone on F.Cu, net GND
- added copper zone on B.Cu, net GNDPWR

Commit message: fix(conch):logo
Other:
- board text added: "2026-0410 conch-v4.0 by jucat"
Changed lines of the file:
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@@
 		(layer "Edge.Cuts")
+	)
+	(gr_text "2026-0410\nconch-v4.0\nby jucat"
+		(at 171.55 73.1 90)
+		(layer "F.SilkS")
+		(effects
+			(font
+				(size 1 1)
+				(thickness 0.15)
+			)
+			(justify left bottom)
+		)
 	)
 	(segment
